Commit message: New multi-camera example

File: tutorials/zed_multi_camera/urdf/urdf.urdf (robot description, URDF)
Before this commit: robot zed_multi_camera, 1 links, 2 joints
Links:
- removed link $(arg multi_link)
- added link zed_front_camera_link
- added link zed_multi_link
- added link zed_rear_camera_link
Joints:
- removed joint ${camera_name_front}_camera_joint
- removed joint ${camera_name_rear}_camera_joint
- added joint zed_front_camera_joint: type fixed, parent zed_front_camera_link, child zed_multi_link, origin xyz=0.06 0.0 0.0 rpy=0 0 0
- added joint zed_rear_camera_joint: type fixed, parent zed_multi_link, child zed_rear_camera_link, origin xyz=-0.06 0.0 0.0 rpy=0 0 3.141592653589793
