Commit message: Fix mutli camera example launch and xacro

File: tutorials/zed_multi_camera/urdf/zed_multi.urdf.xacro (robot description, xacro)
@@ -48,5 +48,5 @@
       <parent link="$(arg camera_name_0)_camera_link"/>
       <child link="$(arg multi_link)"/>
-      <origin xyz="0.06 0.0 0.0" rpy="0 0 0" />
+      <origin xyz="-0.06 0.0 0.0" rpy="0 0 0" />
   </joint>
   <!-- Define the position of the rear camera with respect to the reference link -->
